File: pcb/gingham.sch (KiCad schematic (older format))
At the start: 169 parts, among them J1 Molex-0548190519, J2 ISP, J3 I2C, SW1 SW_Push, SW10 SW_Push, SW11 SW_Push, SW12 SW_Push, SW13 SW_Push, SW14 SW_Push, SW15 SW_Push, SW16 SW_Push, SW17 SW_Push, SW18 SW_Push, SW19 SW_Push, SW2 SW_Push, SW20 SW_Push, SW21 SW_Push, SW22 SW_Push, SW23 SW_Push, SW24 SW_Push, SW25 SW_Push, SW26 SW_Push, SW27 SW_Push, SW28 SW_Push, SW29 SW_Push, SW3 SW_Push, SW30 SW_Push, SW31 SW_Push, SW32 SW_Push, SW33 SW_Push, SW34 SW_Push, SW35 SW_Push, SW36 SW_Push, SW37 SW_Push, SW38 SW_Push, SW39 SW_Push, SW4 SW_Push, SW40 SW_Push, SW41 SW_Push, SW42 SW_Push, SW43 SW_Push, SW44 SW_Push, SW45 SW_Push, SW46 SW_Push, SW47 SW_Push, SW48 SW_Push, SW49 SW_Push, SW5 SW_Push, SW50 SW_Push, SW51 SW_Push, SW52 SW_Push, SW53 SW_Push, SW54 SW_Push, SW55 SW_Push, SW56 SW_Push, SW57 SW_Push, SW58 SW_Push, SW59 SW_Push, SW6 SW_Push, SW60 SW_Push, SW61 SW_Push, SW62 SW_Push, SW63 SW_Push, SW64 SW_Push, SW65 SW_Push, SW66 SW_Push, SW67 SW_Push, SW68 RESET, SW69 BOOT, SW7 SW_Push, SW70 SW_Push, SW71 SW_Push, SW8 SW_Push, SW9 SW_Push, U1 ATMEGA328-PU, U2 MCP23008-E_P, Y1 16MHz

Commit message: Gingaham
Other:
- note added: "Address: 0x20"
Changed lines of the file:
@@
 EESchema Schematic File Version 4
+LIBS:tartan-cache
 EELAYER 29 0
 EELAYER END
@@
 encoding utf-8
 Sheet 1 1
-Title "Tartan"
+Title "Gingham"
 Date "2019-04-18"
 Rev "V1.0"
@@
 Wire Wire Line
 	12625 2975 12625 2275
-Text Label 7425 2575 2    50   ~ 6
+Text Label 7425 2575 2    50   ~ 10
 ROW1
-Text Label 7425 3275 2    50   ~ 6
+Text Label 7425 3275 2    50   ~ 10
 ROW2
-Text Label 7625 1175 1    50   ~ 6
+Text Label 7625 1175 1    50   ~ 10
 COL0
-Text Label 8125 1175 1    50   ~ 6
+Text Label 8125 1175 1    50   ~ 10
 COL1
-Text Label 8625 1175 1    50   ~ 6
+Text Label 8625 1175 1    50   ~ 10
 COL2
-Text Label 9125 1175 1    50   ~ 6
+Text Label 9125 1175 1    50   ~ 10
 COL3
-Text Label 9625 1175 1    50   ~ 6
+Text Label 9625 1175 1    50   ~ 10
 COL4
-Text Label 10125 1175 1    50   ~ 6
+Text Label 10125 1175 1    50   ~ 10
 COL5
-Text Label 10625 1175 1    50   ~ 6
+Text Label 10625 1175 1    50   ~ 10
 COL6
-Text Label 11125 1175 1    50   ~ 6
+Text Label 11125 1175 1    50   ~ 10
 COL7
-Text Label 11625 1175 1    50   ~ 6
+Text Label 11625 1175 1    50   ~ 10
 COL8
-Text Label 12125 1175 1    50   ~ 6
+Text Label 12125 1175 1    50   ~ 10
 COL9
-Text Label 12625 1175 1    50   ~ 6
+Text Label 12625 1175 1    50   ~ 10
 COL10
 $Comp
@@
 	1    0    0    -1
 $EndComp
-Text Label 3275 1725 0    50   ~ 6
+Text Label 3275 1725 0    50   ~ 10
 USB_D+
-Text Label 3275 1625 0    50   ~ 6
+Text Label 3275 1625 0    50   ~ 10
 USB_D-
 Wire Wire Line
@@
 Wire Wire Line
 	2725 6325 2825 6325
-Text Label 2825 6225 0    50   ~ 6
+Text Label 2825 6225 0    50   ~ 10
 USB_D+
-Text Label 2825 6325 0    50   ~ 6
+Text Label 2825 6325 0    50   ~ 10
 USB_D-
-Text Label 2825 5825 0    50   ~ 6
+Text Label 2825 5825 0    50   ~ 10
 RESET
-Text Label 2825 5325 0    50   ~ 6
+Text Label 2825 5325 0    50   ~ 10
 ROW3
 $Comp
@@
 	1    0    0    -1
 $EndComp
-Text Label 4525 5025 2    50   ~ 6
+Text Label 4525 5025 2    50   ~ 10
 RESET
 Wire Wire Line
@@
 Wire Wire Line
 	2725 6625 2825 6625
-Text Label 2925 8425 0    50   ~ 6
+Text Label 2925 8425 0    50   ~ 10
 COL0
-Text Label 2825 6425 0    50   ~ 6
+Text Label 2825 6425 0    50   ~ 10
 COL1
-Text Label 2825 5225 0    50   ~ 6
+Text Label 2825 5225 0    50   ~ 10
 COL2
-Text Label 2825 4825 0    50   ~ 6
+Text Label 2825 4825 0    50   ~ 10
 COL3
-Text Label 7425 1875 2    50   ~ 6
+Text Label 7425 1875 2    50   ~ 10
 ROW0
-Text Label 2825 5525 0    50   ~ 6
+Text Label 2825 5525 0    50   ~ 10
 ROW1
-Text Label 2825 6025 0    50   ~ 6
+Text Label 2825 6025 0    50   ~ 10
 ROW0
-Text Label 2825 6125 0    50   ~ 6
+Text Label 2825 6125 0    50   ~ 10
 ROW2
 Wire Wire Line
@@
 Wire Wire Line
 	2725 4525 2825 4525
-Text Label 2825 6525 0    50   ~ 6
+Text Label 2825 6525 0    50   ~ 10
 COL4
-Text Label 2825 4725 0    50   ~ 6
+Text Label 2825 4725 0    50   ~ 10
 COL5
-Text Label 2825 6625 0    50   ~ 6
+Text Label 2825 6625 0    50   ~ 10
 COL6
 Wire Wire Line
@@
 Wire Wire Line
 	2725 5725 2825 5725
-Text Label 2825 4425 0    50   ~ 6
+Text Label 2825 4425 0    50   ~ 10
 COL7
-Text Label 2825 4325 0    50   ~ 6
+Text Label 2825 4325 0    50   ~ 10
 COL8
-Text Label 2825 4525 0    50   ~ 6
+Text Label 2825 4525 0    50   ~ 10
 COL9
-Text Label 2825 6725 0    50   ~ 6
+Text Label 2825 6725 0    50   ~ 10
 COL10
-Text Label 2825 4625 0    50   ~ 6
+Text Label 2825 4625 0    50   ~ 10
 COL11
 Wire Wire Line
@@
 Wire Wire Line
 	2725 6125 2825 6125
-Text Label 7425 3975 2    50   ~ 6
+Text Label 7425 3975 2    50   ~ 10
 ROW3
 $Comp
@@
 $EndComp
 NoConn ~ 1525 4325
-Text Label 2825 5625 0    50   ~ 6
+Text Label 2825 5625 0    50   ~ 10
 i2c_SDA
 Wire Wire Line
 	4425 6425 4425 6525
-Text Label 2825 5725 0    50   ~ 6
+Text Label 2825 5725 0    50   ~ 10
 i2c_SCL
 Wire Wire Line
@@
 Wire Wire Line
 	1425 8425 1400 8425
-Text Label 900  8525 2    50   ~ 6
+Text Label 900  8525 2    50   ~ 10
 i2c_SCL
-Text Label 900  8425 2    50   ~ 6
+Text Label 900  8425 2    50   ~ 10
 i2c_SDA
 Wire Wire Line
@@
 Wire Wire Line
 	13025 1875 13525 1875
-Text Label 13125 1175 1    50   ~ 6
+Text Label 13125 1175 1    50   ~ 10
 COL11
 Wire Wire Line
@@
 Wire Wire Line
 	13525 1875 14025 1875
-Text Label 13625 1175 1    50   ~ 6
+Text Label 13625 1175 1    50   ~ 10
 COL12
 Wire Wire Line
@@
 Wire Wire Line
 	14025 1875 14525 1875
-Text Label 14125 1175 1    50   ~ 6
+Text Label 14125 1175 1    50   ~ 10
 COL13
 Connection ~ 14125 2975
@@
 Wire Wire Line
 	12625 4375 12625 3675
-Text Label 7425 4675 2    50   ~ 6
+Text Label 7425 4675 2    50   ~ 10
 ROW4
 Wire Wire Line
@@
 	2125 1925 2125 2200
 Connection ~ 2125 1925
-Text Label 2825 5425 0    50   ~ 6
+Text Label 2825 5425 0    50   ~ 10
 ROW4
 Wire Wire Line
 	2825 8425 2925 8425
-Text Label 2925 8525 0    50   ~ 6
+Text Label 2925 8525 0    50   ~ 10
 COL13
 Wire Wire Line
 	2825 8525 2925 8525
-Text Label 2925 8625 0    50   ~ 6
+Text Label 2925 8625 0    50   ~ 10
 COL12
 Wire Wire Line
@@
 Wire Notes Line
 	475  2500 5725 2500
-Text Notes 4725 2350 0    200  ~ 6
+Text Notes 4725 2350 0    200  ~ 40
 Power
 Wire Notes Line
 	5725 5300 16050 5300
-Text Notes 15125 5250 0    200  ~ 6
+Text Notes 15125 5250 0    200  ~ 40
 Matrix
 Wire Notes Line
@@
 Wire Notes Line
 	500  7500 5725 7500
-Text Notes 5025 7425 0    200  ~ 6
+Text Notes 5025 7425 0    200  ~ 40
 MCU
-Text Notes 3500 11100 0    200  ~ 6
+Text Notes 3500 11100 0    200  ~ 40
 Port Expander
 $Comp
@@
 Wire Wire Line
 	4650 3575 4725 3575
-Text Label 4650 3475 2    50   ~ 6
+Text Label 4650 3475 2    50   ~ 10
 i2c_SCL
 Wire Wire Line
 	4650 3475 4725 3475
-Text Label 4650 3375 2    50   ~ 6
+Text Label 4650 3375 2    50   ~ 10
 i2c_SDA
 Wire Wire Line
 	4650 3375 4725 3375
+Text Notes 2675 10100 0    50   ~ 0
+Address: 0x20
 $EndSCHEMATC
