File: pcb/gingham_bottom.kicad_pcb (KiCad board)
At the start: 2 copper layers, 285.8 x 123.8 mm, 10 parts

Commit message: Gingaham
Parts:
- removed tartan_katakana: G***, tartan:tartan_katakana
- added H5: M2, MountingHole:MountingHole_2.2mm_M2_DIN965_Pad, F.Cu at (71.4, 95.2)
- added svg2mod: G***, tartan:gingham_katakana, B.Cu at (189.0, 123.0)
Other:
- board text added: "Designed and assembled by Yiancar in Cambridge, UK Gingham V1.0 Inspired by Plaid"
- board text removed: "Designed and assembled by Yiancar in Cambridge, UK Tartar V1.0 Inspired by Plaid"

Commit message: Relocate middle screwmounts
Parts:
- moved H10 7.49 mm to (188.1, 159.5)
- moved H9 3.48 mm to (188.1, 92.7)
Changed lines of the file:
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@@
   )
   (module MountingHole:MountingHole_2.2mm_M2_DIN965_Pad (layer F.Cu)
-    (at 190.49375 95.24375)
+    (at 188.125 92.7)
     (descr "Mounting Hole 2.2mm, M2, DIN965")
     (tags "mounting hole 2.2mm m2 din965")
@@
   )
   (module MountingHole:MountingHole_2.2mm_M2_DIN965_Pad (layer F.Cu)
-    (at 190.49375 152.39375)
+    (at 188.125 159.5)
     (descr "Mounting Hole 2.2mm, M2, DIN965")
     (tags "mounting hole 2.2mm m2 din965")
